File: kicad/quadrant.sch (KiCad schematic (older format))
At the start: 20 parts, among them J1 Conn_01x06, J2 USB_B_Micro, Q1 2N2219, U1 STM32F070F6Px, U2 AZ1117-3.3

Commit message: update schematic for rev 2
Parts:
- removed D1: TCRT5000, quadrant:TCRT5000, symbol quadrant:TCRT5000
- removed Q1: 2N2219, Package_TO_SOT_THT:TO-92, symbol Transistor_BJT:2N2219
- added C2, C3: 20 pF, symbol Device:C
- added C4: 10 uF, symbol Device:C
- added C5: 22 uF, symbol Device:C
- added D4: TCRT5000, quadrant:TCRT5000, symbol quadrant:TCRT5000
- added D5: LED, symbol Device:LED
- added Q1, Q2, Q3, Q4: NPN, symbol Device:Q_NPN_BCE
- added R11, R14: 1k, Resistor_SMD:R_1206_3216Metric_Pad1.42x1.75mm_HandSolder, symbol Device:R
- added R12: 33k, Resistor_SMD:R_1206_3216Metric_Pad1.42x1.75mm_HandSolder, symbol Device:R
- added R13: 33, Resistor_SMD:R_1206_3216Metric_Pad1.42x1.75mm_HandSolder, symbol Device:R
- added Y1: 8 MHz, symbol Device:Crystal
- R1: value 33k -> 68; footprint Resistor_SMD:R_1206_3216Metric_Pad1.42x1.75mm_HandSolder -> (none)
- R2: value 33 -> 33k
- R5: value 33k -> 33
- R6: value 33 -> 1k
- renumbered D4 to D1
Connections:
- net labels added: ADC_IN0, ADC_IN2, ADC_IN4, ADC_IN6, PA1, PA3, PA5, PA7
- wire segments 61 -> 64
- no-connect marks 8 -> 2
Other:
- moved on the sheet: U2

Commit message: associate footprints with schematic symbols
Parts:
- C1: footprint Capacitor_SMD:C_1206_3216Metric_Pad1.42x1.75mm_HandSolder -> Capacitor_SMD:C_0805_2012Metric_Pad1.15x1.40mm_HandSolder
- C2, C3, C4, C5: footprint (none) -> Capacitor_SMD:C_0805_2012Metric_Pad1.15x1.40mm_HandSolder
- D5: footprint (none) -> LED_SMD:LED_1206_3216Metric_Pad1.42x1.75mm_HandSolder
- Q1, Q2, Q3, Q4: footprint (none) -> Package_TO_SOT_SMD:SOT-23
- R1: footprint (none) -> Resistor_SMD:R_0805_2012Metric_Pad1.15x1.40mm_HandSolder
- R10, R11, R12, R13, R14, R2, R3, R4, R5, R6, R7, R8, R9: footprint Resistor_SMD:R_1206_3216Metric_Pad1.42x1.75mm_HandSolder -> Resistor_SMD:R_0805_2012Metric_Pad1.15x1.40mm_HandSolder
- Y1: footprint (none) -> Crystal:Crystal_HC49-U_Vertical
Changed lines of the file:
@@
 F 0 "R9" H 8420 2346 50  0000 L CNN
 F 1 "1k" H 8420 2255 50  0000 L CNN
-F 2 "Resistor_SMD:R_1206_3216Metric_Pad1.42x1.75mm_HandSolder" V 8280 2300 50  0001 C CNN
+F 2 "Resistor_SMD:R_0805_2012Metric_Pad1.15x1.40mm_HandSolder" V 8280 2300 50  0001 C CNN
 F 3 "~" H 8350 2300 50  0001 C CNN
 	1    8350 2300
@@
 F 0 "R3" H 7720 1196 50  0000 L CNN
 F 1 "33k" H 7720 1105 50  0000 L CNN
-F 2 "Resistor_SMD:R_1206_3216Metric_Pad1.42x1.75mm_HandSolder" V 7580 1150 50  0001 C CNN
+F 2 "Resistor_SMD:R_0805_2012Metric_Pad1.15x1.40mm_HandSolder" V 7580 1150 50  0001 C CNN
 F 3 "~" H 7650 1150 50  0001 C CNN
 	1    7650 1150
@@
 F 0 "R4" H 7970 1196 50  0000 L CNN
 F 1 "33" H 7970 1105 50  0000 L CNN
-F 2 "Resistor_SMD:R_1206_3216Metric_Pad1.42x1.75mm_HandSolder" V 7830 1150 50  0001 C CNN
+F 2 "Resistor_SMD:R_0805_2012Metric_Pad1.15x1.40mm_HandSolder" V 7830 1150 50  0001 C CNN
 F 3 "~" H 7900 1150 50  0001 C CNN
 	1    7900 1150
@@
 F 0 "C1" V 2848 4650 50  0000 C CNN
 F 1 "100 nF" V 2939 4650 50  0000 C CNN
-F 2 "Capacitor_SMD:C_1206_3216Metric_Pad1.42x1.75mm_HandSolder" H 3138 4500 50  0001 C CNN
+F 2 "Capacitor_SMD:C_0805_2012Metric_Pad1.15x1.40mm_HandSolder" H 3138 4500 50  0001 C CNN
 F 3 "~" H 3100 4650 50  0001 C CNN
 	1    3100 4650
@@
 F 0 "R10" H 2530 5354 50  0000 R CNN
 F 1 "10k" H 2530 5445 50  0000 R CNN
-F 2 "Resistor_SMD:R_1206_3216Metric_Pad1.42x1.75mm_HandSolder" V 2530 5400 50  0001 C CNN
+F 2 "Resistor_SMD:R_0805_2012Metric_Pad1.15x1.40mm_HandSolder" V 2530 5400 50  0001 C CNN
 F 3 "~" H 2600 5400 50  0001 C CNN
 	1    2600 5400
@@
 F 0 "C5" H 3965 3496 50  0000 L CNN
 F 1 "22 uF" H 3965 3405 50  0000 L CNN
-F 2 "" H 3888 3300 50  0001 C CNN
+F 2 "Capacitor_SMD:C_0805_2012Metric_Pad1.15x1.40mm_HandSolder" H 3888 3300 50  0001 C CNN
 F 3 "~" H 3850 3450 50  0001 C CNN
 	1    3850 3450
@@
 F 0 "C4" H 2915 3496 50  0000 L CNN
 F 1 "10 uF" H 2915 3405 50  0000 L CNN
-F 2 "" H 2838 3300 50  0001 C CNN
+F 2 "Capacitor_SMD:C_0805_2012Metric_Pad1.15x1.40mm_HandSolder" H 2838 3300 50  0001 C CNN
 F 3 "~" H 2800 3450 50  0001 C CNN
 	1    2800 3450
@@
 F 0 "Y1" V 2204 6131 50  0000 L CNN
 F 1 "8 MHz" V 2295 6131 50  0000 L CNN
-F 2 "" H 2250 6000 50  0001 C CNN
+F 2 "Crystal:Crystal_HC49-U_Vertical" H 2250 6000 50  0001 C CNN
 F 3 "~" H 2250 6000 50  0001 C CNN
 	1    2250 6000
@@
 F 0 "C2" V 1698 5850 50  0000 C CNN
 F 1 "20 pF" V 1789 5850 50  0000 C CNN
-F 2 "" H 1988 5700 50  0001 C CNN
+F 2 "Capacitor_SMD:C_0805_2012Metric_Pad1.15x1.40mm_HandSolder" H 1988 5700 50  0001 C CNN
 F 3 "~" H 1950 5850 50  0001 C CNN
 	1    1950 5850
@@
 F 0 "C3" V 2100 6150 50  0000 C CNN
 F 1 "20 pF" V 2200 6150 50  0000 C CNN
-F 2 "" H 1988 6000 50  0001 C CNN
+F 2 "Capacitor_SMD:C_0805_2012Metric_Pad1.15x1.40mm_HandSolder" H 1988 6000 50  0001 C CNN
 F 3 "~" H 1950 6150 50  0001 C CNN
 	1    1950 6150
@@
 F 0 "Q1" H 7850 2400 50  0000 L CNN
 F 1 "NPN" H 7800 2150 50  0000 L CNN
-F 2 "" H 8200 2400 50  0001 C CNN
+F 2 "Package_TO_SOT_SMD:SOT-23" H 8200 2400 50  0001 C CNN
 F 3 "~" H 8000 2300 50  0001 C CNN
 	1    8000 2300
@@
 F 0 "R6" H 6720 3946 50  0000 L CNN
 F 1 "1k" H 6720 3855 50  0000 L CNN
-F 2 "Resistor_SMD:R_1206_3216Metric_Pad1.42x1.75mm_HandSolder" V 6580 3900 50  0001 C CNN
+F 2 "Resistor_SMD:R_0805_2012Metric_Pad1.15x1.40mm_HandSolder" V 6580 3900 50  0001 C CNN
 F 3 "~" H 6650 3900 50  0001 C CNN
 	1    6650 3900
@@
 F 0 "R2" H 6020 2796 50  0000 L CNN
 F 1 "33k" H 6020 2705 50  0000 L CNN
-F 2 "Resistor_SMD:R_1206_3216Metric_Pad1.42x1.75mm_HandSolder" V 5880 2750 50  0001 C CNN
+F 2 "Resistor_SMD:R_0805_2012Metric_Pad1.15x1.40mm_HandSolder" V 5880 2750 50  0001 C CNN
 F 3 "~" H 5950 2750 50  0001 C CNN
 	1    5950 2750
@@
 F 0 "R5" H 6270 2796 50  0000 L CNN
 F 1 "33" H 6270 2705 50  0000 L CNN
-F 2 "Resistor_SMD:R_1206_3216Metric_Pad1.42x1.75mm_HandSolder" V 6130 2750 50  0001 C CNN
+F 2 "Resistor_SMD:R_0805_2012Metric_Pad1.15x1.40mm_HandSolder" V 6130 2750 50  0001 C CNN
 F 3 "~" H 6200 2750 50  0001 C CNN
 	1    6200 2750
@@
 F 0 "Q4" H 6150 4000 50  0000 L CNN
 F 1 "NPN" H 6100 3750 50  0000 L CNN
-F 2 "" H 6500 4000 50  0001 C CNN
+F 2 "Package_TO_SOT_SMD:SOT-23" H 6500 4000 50  0001 C CNN
 F 3 "~" H 6300 3900 50  0001 C CNN
 	1    6300 3900
@@
 F 0 "R11" H 8420 5696 50  0000 L CNN
 F 1 "1k" H 8420 5605 50  0000 L CNN
-F 2 "Resistor_SMD:R_1206_3216Metric_Pad1.42x1.75mm_HandSolder" V 8280 5650 50  0001 C CNN
+F 2 "Resistor_SMD:R_0805_2012Metric_Pad1.15x1.40mm_HandSolder" V 8280 5650 50  0001 C CNN
 F 3 "~" H 8350 5650 50  0001 C CNN
 	1    8350 5650
@@
 F 0 "R7" H 7720 4546 50  0000 L CNN
 F 1 "33k" H 7720 4455 50  0000 L CNN
-F 2 "Resistor_SMD:R_1206_3216Metric_Pad1.42x1.75mm_HandSolder" V 7580 4500 50  0001 C CNN
+F 2 "Resistor_SMD:R_0805_2012Metric_Pad1.15x1.40mm_HandSolder" V 7580 4500 50  0001 C CNN
 F 3 "~" H 7650 4500 50  0001 C CNN
 	1    7650 4500
@@
 F 0 "R8" H 7970 4546 50  0000 L CNN
 F 1 "33" H 7970 4455 50  0000 L CNN
-F 2 "Resistor_SMD:R_1206_3216Metric_Pad1.42x1.75mm_HandSolder" V 7830 4500 50  0001 C CNN
+F 2 "Resistor_SMD:R_0805_2012Metric_Pad1.15x1.40mm_HandSolder" V 7830 4500 50  0001 C CNN
 F 3 "~" H 7900 4500 50  0001 C CNN
 	1    7900 4500
@@
 F 0 "Q3" H 7850 5750 50  0000 L CNN
 F 1 "NPN" H 7800 5500 50  0000 L CNN
-F 2 "" H 8200 5750 50  0001 C CNN
+F 2 "Package_TO_SOT_SMD:SOT-23" H 8200 5750 50  0001 C CNN
 F 3 "~" H 8000 5650 50  0001 C CNN
 	1    8000 5650
@@
 F 0 "R14" H 10170 3946 50  0000 L CNN
 F 1 "1k" H 10170 3855 50  0000 L CNN
-F 2 "Resistor_SMD:R_1206_3216Metric_Pad1.42x1.75mm_HandSolder" V 10030 3900 50  0001 C CNN
+F 2 "Resistor_SMD:R_0805_2012Metric_Pad1.15x1.40mm_HandSolder" V 10030 3900 50  0001 C CNN
 F 3 "~" H 10100 3900 50  0001 C CNN
 	1    10100 3900
@@
 F 0 "R12" H 9470 2796 50  0000 L CNN
 F 1 "33k" H 9470 2705 50  0000 L CNN
-F 2 "Resistor_SMD:R_1206_3216Metric_Pad1.42x1.75mm_HandSolder" V 9330 2750 50  0001 C CNN
+F 2 "Resistor_SMD:R_0805_2012Metric_Pad1.15x1.40mm_HandSolder" V 9330 2750 50  0001 C CNN
 F 3 "~" H 9400 2750 50  0001 C CNN
 	1    9400 2750
@@
 F 0 "R13" H 9720 2796 50  0000 L CNN
 F 1 "33" H 9720 2705 50  0000 L CNN
-F 2 "Resistor_SMD:R_1206_3216Metric_Pad1.42x1.75mm_HandSolder" V 9580 2750 50  0001 C CNN
+F 2 "Resistor_SMD:R_0805_2012Metric_Pad1.15x1.40mm_HandSolder" V 9580 2750 50  0001 C CNN
 F 3 "~" H 9650 2750 50  0001 C CNN
 	1    9650 2750
@@
 F 0 "Q2" H 9600 4000 50  0000 L CNN
 F 1 "NPN" H 9550 3750 50  0000 L CNN
-F 2 "" H 9950 4000 50  0001 C CNN
+F 2 "Package_TO_SOT_SMD:SOT-23" H 9950 4000 50  0001 C CNN
 F 3 "~" H 9750 3900 50  0001 C CNN
 	1    9750 3900
@@
 F 0 "D5" H 2691 6766 50  0000 C CNN
 F 1 "LED" H 2691 6675 50  0000 C CNN
-F 2 "" H 2700 6550 50  0001 C CNN
+F 2 "LED_SMD:LED_1206_3216Metric_Pad1.42x1.75mm_HandSolder" H 2700 6550 50  0001 C CNN
 F 3 "~" H 2700 6550 50  0001 C CNN
 	1    2700 6550
@@
 F 0 "R1" V 2143 6550 50  0000 C CNN
 F 1 "68" V 2234 6550 50  0000 C CNN
-F 2 "" V 2280 6550 50  0001 C CNN
+F 2 "Resistor_SMD:R_0805_2012Metric_Pad1.15x1.40mm_HandSolder" V 2280 6550 50  0001 C CNN
 F 3 "~" H 2350 6550 50  0001 C CNN
 	1    2350 6550

Commit message: change NPN schematic symbols from BCE to BEC
Parts:
- Q1, Q2, Q3, Q4: symbol Device:Q_NPN_BCE -> Device:Q_NPN_BEC
Changed lines of the file:
@@
 	7650 2500 7650 2650
 $Comp
-L Device:Q_NPN_BCE Q1
+L Device:Q_NPN_BEC Q1
 U 1 1 5BD10622
 P 8000 2300
@@
 	5950 4100 5950 4250
 $Comp
-L Device:Q_NPN_BCE Q4
+L Device:Q_NPN_BEC Q4
 U 1 1 5BD13833
 P 6300 3900
@@
 	7650 5850 7650 6000
 $Comp
-L Device:Q_NPN_BCE Q3
+L Device:Q_NPN_BEC Q3
 U 1 1 5BD1467A
 P 8000 5650
@@
 	9400 4100 9400 4250
 $Comp
-L Device:Q_NPN_BCE Q2
+L Device:Q_NPN_BEC Q2
 U 1 1 5BD146B7
 P 9750 3900
