File: kicad/quadrant.sch (KiCad schematic (older format))
At the start: 33 parts, among them J1 Conn_01x06, J2 USB_B_Micro, Q1 NPN, Q2 NPN, Q3 NPN, Q4 NPN, U1 STM32F070F6Px, U2 AZ1117-3.3, Y1 8 MHz

Commit message: schematic: changed load capacitors on crystal oscillator to 18 pF
Parts:
- C2, C3: value 20 pF -> 18 pF
Changed lines of the file:
@@
 Sheet 1 1
 Title "Quadrant Board"
-Date "2018-10-22"
+Date "2018-11-16"
 Rev "2"
 Comp "Chris Chronopoulos"
@@
 P 1950 5850
 F 0 "C2" V 1698 5850 50  0000 C CNN
-F 1 "20 pF" V 1789 5850 50  0000 C CNN
+F 1 "18 pF" V 1789 5850 50  0000 C CNN
 F 2 "Capacitor_SMD:C_0805_2012Metric_Pad1.15x1.40mm_HandSolder" H 1988 5700 50  0001 C CNN
 F 3 "~" H 1950 5850 50  0001 C CNN
@@
 P 1950 6150
 F 0 "C3" V 2100 6150 50  0000 C CNN
-F 1 "20 pF" V 2200 6150 50  0000 C CNN
+F 1 "18 pF" V 2200 6150 50  0000 C CNN
 F 2 "Capacitor_SMD:C_0805_2012Metric_Pad1.15x1.40mm_HandSolder" H 1988 6000 50  0001 C CNN
 F 3 "~" H 1950 6150 50  0001 C CNN

Commit message: quadrant.sch: first pass at a rev 3 schematic
Parts:
- removed C1: 100 nF, Capacitor_SMD:C_0805_2012Metric_Pad1.15x1.40mm_HandSolder, symbol Device:C
- removed C2, C3: 18 pF, Capacitor_SMD:C_0805_2012Metric_Pad1.15x1.40mm_HandSolder, symbol Device:C
- removed C4: 10 uF, Capacitor_SMD:C_0805_2012Metric_Pad1.15x1.40mm_HandSolder, symbol Device:C
- removed C5: 22 uF, Capacitor_SMD:C_0805_2012Metric_Pad1.15x1.40mm_HandSolder, symbol Device:C
- removed D1, D2, D3, D4: TCRT5000, quadrant:TCRT5000, symbol quadrant:TCRT5000
- removed D5: LED, LED_SMD:LED_1206_3216Metric_Pad1.42x1.75mm_HandSolder, symbol Device:LED
- removed Q1, Q2, Q3, Q4: NPN, Package_TO_SOT_SMD:SOT-23, symbol Device:Q_NPN_BEC
- removed R1: 68, Resistor_SMD:R_0805_2012Metric_Pad1.15x1.40mm_HandSolder, symbol Device:R
- removed R10: 10k, Resistor_SMD:R_0805_2012Metric_Pad1.15x1.40mm_HandSolder, symbol Device:R
- removed R11, R14, R6, R9: 1k, Resistor_SMD:R_0805_2012Metric_Pad1.15x1.40mm_HandSolder, symbol Device:R
- removed R12, R2, R3, R7: 33k, Resistor_SMD:R_0805_2012Metric_Pad1.15x1.40mm_HandSolder, symbol Device:R
- removed R13, R4, R5, R8: 33, Resistor_SMD:R_0805_2012Metric_Pad1.15x1.40mm_HandSolder, symbol Device:R
- removed U1: STM32F070F6Px, Package_SO:TSSOP-20_4.4x6.5mm_P0.65mm, symbol MCU_ST_STM32F0:STM32F070F6Px
- removed U2: AZ1117-3.3, Package_TO_SOT_SMD:SOT-89-3_Handsoldering, symbol Regulator_Linear:AZ1117-3.3
- removed Y1: 8 MHz, Crystal:Crystal_HC49-U_Vertical, symbol Device:Crystal
- added C? (x4): 0.1uF, symbol Device:C
- added C?: 100 nF, Capacitor_SMD:C_0805_2012Metric_Pad1.15x1.40mm_HandSolder, symbol Device:C
- added C? (x2): 18 pF, Capacitor_SMD:C_0805_2012Metric_Pad1.15x1.40mm_HandSolder, symbol Device:C
- added C? (x2): 1uF, symbol Device:C
- added C?: 10uF, symbol Device:C
- added R?: 10k, Resistor_SMD:R_0805_2012Metric_Pad1.15x1.40mm_HandSolder, symbol Device:R
- added R? (x2): R, symbol Device:R
- added U? (x4): VL6180X, symbol quadrant:VL6180X
- added U?: STM32F070CBTx, Package_QFP:LQFP-48_7x7mm_P0.5mm, symbol MCU_ST_STM32F0:STM32F070CBTx
- added U?: MIC5356-MGYML, Package_DFN_QFN:MLF-8-1EP_3x3mm_P0.65mm_EP1.55x2.3mm_ThermalVias, symbol Regulator_Linear:MIC5356-MGYML
- added Y?: 8 MHz, Crystal:Crystal_HC49-U_Vertical, symbol Device:Crystal
Connections:
- net labels added: +2V8, +3V3, SCL, SDA
- net labels removed: ADC_IN0, ADC_IN2, ADC_IN4, ADC_IN6, PA1, PA3, PA5, PA7
- wire segments 64 -> 112

Commit message: quadrant.sch: add LEDs, and update symbol for LDO
Parts:
- removed U?: MIC5356-MGYML, Package_DFN_QFN:MLF-8-1EP_3x3mm_P0.65mm_EP1.55x2.3mm_ThermalVias, symbol Regulator_Linear:MIC5356-MGYML
- added C?: 10uF, symbol Device:C
- added D? (x4): LED, symbol Device:LED
- added R? (x4): R, symbol Device:R
- added U?: MIC5399-SMYMX, symbol quadrant:MIC5399-SMYMX
- C?: value 100 nF -> 0.1 uF
- R? (x2): value R -> 4.7k
Connections:
- wire segments 112 -> 128

Commit message: quadrant.sch: annotate symbols
Parts:
- gave numbers to parts that had none: 29

Commit message: quadrant.sch: assign footprints
Parts:
- C1, C2, C3, C4, C5, C6, C7, C8: footprint (none) -> Capacitor_SMD:C_0805_2012Metric_Pad1.15x1.40mm_HandSolder
- D1, D2, D3, D4: footprint (none) -> LED_SMD:LED_1206_3216Metric_Pad1.42x1.75mm_HandSolder
- R2, R3, R4, R5, R6, R7: footprint (none) -> Resistor_SMD:R_0805_2012Metric_Pad1.15x1.40mm_HandSolder
- U1, U3, U4, U5: footprint (none) -> quadrant:VL6180X
Changed lines of the file:
@@
 F 0 "U3" H 3400 4725 50  0000 C CNN
 F 1 "VL6180X" H 3400 4634 50  0000 C CNN
-F 2 "" H 3250 4300 50  0001 C CNN
+F 2 "quadrant:VL6180X" H 3250 4300 50  0001 C CNN
 F 3 "" H 3250 4300 50  0001 C CNN
 	1    3400 4300
@@
 F 0 "C6" V 4198 4300 50  0000 C CNN
 F 1 "0.1uF" V 4289 4300 50  0000 C CNN
-F 2 "" H 4488 4150 50  0001 C CNN
+F 2 "Capacitor_SMD:C_0805_2012Metric_Pad1.15x1.40mm_HandSolder" H 4488 4150 50  0001 C CNN
 F 3 "~" H 4450 4300 50  0001 C CNN
 	1    4450 4300
@@
 F 0 "C4" H 3965 2796 50  0000 L CNN
 F 1 "1uF" H 3965 2705 50  0000 L CNN
-F 2 "" H 3888 2600 50  0001 C CNN
+F 2 "Capacitor_SMD:C_0805_2012Metric_Pad1.15x1.40mm_HandSolder" H 3888 2600 50  0001 C CNN
 F 3 "~" H 3850 2750 50  0001 C CNN
 	1    3850 2750
@@
 F 0 "C5" H 4365 2796 50  0000 L CNN
 F 1 "1uF" H 4365 2705 50  0000 L CNN
-F 2 "" H 4288 2600 50  0001 C CNN
+F 2 "Capacitor_SMD:C_0805_2012Metric_Pad1.15x1.40mm_HandSolder" H 4288 2600 50  0001 C CNN
 F 3 "~" H 4250 2750 50  0001 C CNN
 	1    4250 2750
@@
 F 0 "C2" H 2465 2796 50  0000 L CNN
 F 1 "10uF" H 2465 2705 50  0000 L CNN
-F 2 "" H 2388 2600 50  0001 C CNN
+F 2 "Capacitor_SMD:C_0805_2012Metric_Pad1.15x1.40mm_HandSolder" H 2388 2600 50  0001 C CNN
 F 3 "~" H 2350 2750 50  0001 C CNN
 	1    2350 2750
@@
 F 0 "R6" H 9670 4146 50  0000 L CNN
 F 1 "4.7k" H 9670 4055 50  0000 L CNN
-F 2 "" V 9530 4100 50  0001 C CNN
+F 2 "Resistor_SMD:R_0805_2012Metric_Pad1.15x1.40mm_HandSolder" V 9530 4100 50  0001 C CNN
 F 3 "~" H 9600 4100 50  0001 C CNN
 	1    9600 4100
@@
 F 0 "R7" H 9970 4146 50  0000 L CNN
 F 1 "4.7k" H 9970 4055 50  0000 L CNN
-F 2 "" V 9830 4100 50  0001 C CNN
+F 2 "Resistor_SMD:R_0805_2012Metric_Pad1.15x1.40mm_HandSolder" V 9830 4100 50  0001 C CNN
 F 3 "~" H 9900 4100 50  0001 C CNN
 	1    9900 4100
@@
 F 0 "U4" H 3400 7375 50  0000 C CNN
 F 1 "VL6180X" H 3400 7284 50  0000 C CNN
-F 2 "" H 3250 6950 50  0001 C CNN
+F 2 "quadrant:VL6180X" H 3250 6950 50  0001 C CNN
 F 3 "" H 3250 6950 50  0001 C CNN
 	1    3400 6950
@@
 F 0 "C7" V 4198 6950 50  0000 C CNN
 F 1 "0.1uF" V 4289 6950 50  0000 C CNN
-F 2 "" H 4488 6800 50  0001 C CNN
+F 2 "Capacitor_SMD:C_0805_2012Metric_Pad1.15x1.40mm_HandSolder" H 4488 6800 50  0001 C CNN
 F 3 "~" H 4450 6950 50  0001 C CNN
 	1    4450 6950
@@
 F 0 "U1" H 1700 6025 50  0000 C CNN
 F 1 "VL6180X" H 1700 5934 50  0000 C CNN
-F 2 "" H 1550 5600 50  0001 C CNN
+F 2 "quadrant:VL6180X" H 1550 5600 50  0001 C CNN
 F 3 "" H 1550 5600 50  0001 C CNN
 	1    1700 5600
@@
 F 0 "C3" V 2498 5600 50  0000 C CNN
 F 1 "0.1uF" V 2589 5600 50  0000 C CNN
-F 2 "" H 2788 5450 50  0001 C CNN
+F 2 "Capacitor_SMD:C_0805_2012Metric_Pad1.15x1.40mm_HandSolder" H 2788 5450 50  0001 C CNN
 F 3 "~" H 2750 5600 50  0001 C CNN
 	1    2750 5600
@@
 F 0 "U5" H 4900 6025 50  0000 C CNN
 F 1 "VL6180X" H 4900 5934 50  0000 C CNN
-F 2 "" H 4750 5600 50  0001 C CNN
+F 2 "quadrant:VL6180X" H 4750 5600 50  0001 C CNN
 F 3 "" H 4750 5600 50  0001 C CNN
 	1    4900 5600
@@
 F 0 "C8" V 5698 5600 50  0000 C CNN
 F 1 "0.1uF" V 5789 5600 50  0000 C CNN
-F 2 "" H 5988 5450 50  0001 C CNN
+F 2 "Capacitor_SMD:C_0805_2012Metric_Pad1.15x1.40mm_HandSolder" H 5988 5450 50  0001 C CNN
 F 3 "~" H 5950 5600 50  0001 C CNN
 	1    5950 5600
@@
 F 0 "D1" H 7842 3145 50  0000 C CNN
 F 1 "LED" H 7842 3236 50  0000 C CNN
-F 2 "" H 7850 3400 50  0001 C CNN
+F 2 "LED_SMD:LED_1206_3216Metric_Pad1.42x1.75mm_HandSolder" H 7850 3400 50  0001 C CNN
 F 3 "~" H 7850 3400 50  0001 C CNN
 	1    7850 3400
@@
 F 0 "R2" V 7343 3400 50  0000 C CNN
 F 1 "R" V 7434 3400 50  0000 C CNN
-F 2 "" V 7480 3400 50  0001 C CNN
+F 2 "Resistor_SMD:R_0805_2012Metric_Pad1.15x1.40mm_HandSolder" V 7480 3400 50  0001 C CNN
 F 3 "~" H 7550 3400 50  0001 C CNN
 	1    7550 3400
@@
 F 0 "D4" H 7842 4345 50  0000 C CNN
 F 1 "LED" H 7842 4436 50  0000 C CNN
-F 2 "" H 7850 4600 50  0001 C CNN
+F 2 "LED_SMD:LED_1206_3216Metric_Pad1.42x1.75mm_HandSolder" H 7850 4600 50  0001 C CNN
 F 3 "~" H 7850 4600 50  0001 C CNN
 	1    7850 4600
@@
 F 0 "R5" V 7343 4600 50  0000 C CNN
 F 1 "R" V 7434 4600 50  0000 C CNN
-F 2 "" V 7480 4600 50  0001 C CNN
+F 2 "Resistor_SMD:R_0805_2012Metric_Pad1.15x1.40mm_HandSolder" V 7480 4600 50  0001 C CNN
 F 3 "~" H 7550 4600 50  0001 C CNN
 	1    7550 4600
@@
 F 0 "D2" H 7842 3545 50  0000 C CNN
 F 1 "LED" H 7842 3636 50  0000 C CNN
-F 2 "" H 7850 3800 50  0001 C CNN
+F 2 "LED_SMD:LED_1206_3216Metric_Pad1.42x1.75mm_HandSolder" H 7850 3800 50  0001 C CNN
 F 3 "~" H 7850 3800 50  0001 C CNN
 	1    7850 3800
@@
 F 0 "R3" V 7343 3800 50  0000 C CNN
 F 1 "R" V 7434 3800 50  0000 C CNN
-F 2 "" V 7480 3800 50  0001 C CNN
+F 2 "Resistor_SMD:R_0805_2012Metric_Pad1.15x1.40mm_HandSolder" V 7480 3800 50  0001 C CNN
 F 3 "~" H 7550 3800 50  0001 C CNN
 	1    7550 3800
@@
 F 0 "D3" H 7842 3945 50  0000 C CNN
 F 1 "LED" H 7842 4036 50  0000 C CNN
-F 2 "" H 7850 4200 50  0001 C CNN
+F 2 "LED_SMD:LED_1206_3216Metric_Pad1.42x1.75mm_HandSolder" H 7850 4200 50  0001 C CNN
 F 3 "~" H 7850 4200 50  0001 C CNN
 	1    7850 4200
@@
 F 0 "R4" V 7343 4200 50  0000 C CNN
 F 1 "R" V 7434 4200 50  0000 C CNN
-F 2 "" V 7480 4200 50  0001 C CNN
+F 2 "Resistor_SMD:R_0805_2012Metric_Pad1.15x1.40mm_HandSolder" V 7480 4200 50  0001 C CNN
 F 3 "~" H 7550 4200 50  0001 C CNN
 	1    7550 4200
@@
 F 0 "C1" H 2065 2796 50  0000 L CNN
 F 1 "10uF" H 2065 2705 50  0000 L CNN
-F 2 "" H 1988 2600 50  0001 C CNN
+F 2 "Capacitor_SMD:C_0805_2012Metric_Pad1.15x1.40mm_HandSolder" H 1988 2600 50  0001 C CNN
 F 3 "~" H 1950 2750 50  0001 C CNN
 	1    1950 2750

Commit message: quadrant.sch: add 47k pull-ups for VL6180X GPIOs
Parts:
- added R? (x8): 47k, symbol Device:R
Connections:
- wire segments 128 -> 140

Commit message: quadrant.sch: add 4.7uF bypass caps to AVDD_VCSEL on VL6180x
Parts:
- removed C3, C7, C8: 0.1uF, Capacitor_SMD:C_0805_2012Metric_Pad1.15x1.40mm_HandSolder, symbol Device:C
- removed R? (x6): 47k, symbol Device:R
- removed U1, U4, U5: VL6180X, quadrant:VL6180X, symbol quadrant:VL6180X
- added C? (x4): 4.7uF, symbol Device:C
- added C? (x3): 0.1uF, Capacitor_SMD:C_0805_2012Metric_Pad1.15x1.40mm_HandSolder, symbol Device:C
- added R? (x6): 47k, symbol Device:R
- added U? (x3): VL6180X, quadrant:VL6180X, symbol quadrant:VL6180X
Connections:
- wire segments 140 -> 156

Commit message: replace MIC5399 with AP7332
Parts:
- removed C2: 10uF, Capacitor_SMD:C_0805_2012Metric_Pad1.15x1.40mm_HandSolder, symbol Device:C
- removed C5: 1uF, Capacitor_SMD:C_0805_2012Metric_Pad1.15x1.40mm_HandSolder, symbol Device:C
- removed U2: MIC5399-SMYMX, symbol quadrant:MIC5399-SMYMX
- added C8: 1uF, Capacitor_SMD:C_0805_2012Metric_Pad1.15x1.40mm_HandSolder, symbol Device:C
- added U2: AP7332-2833, Package_TO_SOT_SMD:SOT-23-6_Handsoldering, symbol quadrant:AP7332-2833
- C1: value 10uF -> 1uF
- C13, C2, C5, C7: renamed from C?; footprint (none) -> Capacitor_SMD:C_0805_2012Metric_Pad1.15x1.40mm_HandSolder
- R10, R11, R12, R13, R14, R15, R8, R9: renamed from R?; footprint (none) -> Resistor_SMD:R_0805_2012Metric_Pad1.15x1.40mm_HandSolder
- gave numbers to parts that had none: 6
Connections:
- wire segments 156 -> 145
