File: kicad/quadrant.sch (KiCad schematic (older format))
At the start: 42 parts, among them J1 Conn_01x06, J2 USB_B_Micro, U1 VL6180X, U2 AP7332-2833, U3 VL6180X, U4 VL6180X, U5 VL6180X, U6 STM32F070CBTx, Y1 8 MHz

Commit message: add a decoupling cap for each VDD pin
Parts:
- added C15, C16, C17, C18: 0.1 uF, Capacitor_SMD:C_0805_2012Metric_Pad1.15x1.40mm_HandSolder, symbol Device:C
Connections:
- wire segments 145 -> 152
Changed lines of the file:
@@
 L power:GND #PWR0103
 U 1 1 5C36188E
-P 8350 1750
-F 0 "#PWR0103" H 8350 1500 50  0001 C CNN
-F 1 "GND" H 8355 1577 50  0000 C CNN
-F 2 "" H 8350 1750 50  0001 C CNN
-F 3 "" H 8350 1750 50  0001 C CNN
-	1    8350 1750
-	1    0    0    -1
-$EndComp
-Wire Wire Line
-	8350 1750 8350 1700
-Wire Wire Line
-	8350 1700 8450 1700
+P 7100 1900
+F 0 "#PWR0103" H 7100 1650 50  0001 C CNN
+F 1 "GND" H 7105 1727 50  0000 C CNN
+F 2 "" H 7100 1900 50  0001 C CNN
+F 3 "" H 7100 1900 50  0001 C CNN
+	1    7100 1900
+	1    0    0    -1
+$EndComp
 $Comp
 L Device:C C11
 U 1 1 5C361896
-P 8600 1700
-F 0 "C11" V 8348 1700 50  0000 C CNN
-F 1 "0.1 uF" V 8439 1700 50  0000 C CNN
-F 2 "Capacitor_SMD:C_0805_2012Metric_Pad1.15x1.40mm_HandSolder" H 8638 1550 50  0001 C CNN
-F 3 "~" H 8600 1700 50  0001 C CNN
-	1    8600 1700
-	0    1    1    0
-$EndComp
-Wire Wire Line
-	8800 2100 8800 1900
-Wire Wire Line
-	8800 1700 8750 1700
-Wire Wire Line
-	8700 2100 8700 1900
-Wire Wire Line
-	8700 1900 8800 1900
-Connection ~ 8800 1900
-Wire Wire Line
-	8800 1900 8800 1700
-Wire Wire Line
-	8900 2100 8900 1900
-Wire Wire Line
-	8900 1900 8800 1900
-Wire Wire Line
-	9000 2100 9000 1900
-Wire Wire Line
-	9000 1900 8900 1900
-Connection ~ 8900 1900
-Wire Wire Line
-	8600 2100 8600 1900
-Wire Wire Line
-	8600 1900 8700 1900
-Connection ~ 8700 1900
+P 7100 1500
+F 0 "C11" H 7000 1600 50  0000 C CNN
+F 1 "0.1 uF" H 6950 1400 50  0000 C CNN
+F 2 "Capacitor_SMD:C_0805_2012Metric_Pad1.15x1.40mm_HandSolder" H 7138 1350 50  0001 C CNN
+F 3 "~" H 7100 1500 50  0001 C CNN
+	1    7100 1500
+	-1   0    0    1
+$EndComp
 Wire Wire Line
 	6450 2500 8100 2500
@@
 Wire Wire Line
 	7950 2800 7950 3000
-Wire Wire Line
-	8800 1400 8800 1700
-Connection ~ 8800 1700
 Text GLabel 9450 4600 2    50   Input ~ 0
 USBDP
@@
 Wire Wire Line
 	9600 4300 10150 4300
-$Comp
-L power:+3V3 #PWR0117
-U 1 1 5C3A7FD6
-P 8800 1400
-F 0 "#PWR0117" H 8800 1250 50  0001 C CNN
-F 1 "+3V3" H 8815 1573 50  0000 C CNN
-F 2 "" H 8800 1400 50  0001 C CNN
-F 3 "" H 8800 1400 50  0001 C CNN
-	1    8800 1400
-	1    0    0    -1
-$EndComp
 Wire Wire Line
 	3850 4350 4000 4350
@@
 Wire Wire Line
 	2800 2400 2800 2500
+$Comp
+L Device:C C15
+U 1 1 5C4CAAB9
+P 7450 1500
+F 0 "C15" H 7350 1600 50  0000 C CNN
+F 1 "0.1 uF" H 7300 1400 50  0000 C CNN
+F 2 "Capacitor_SMD:C_0805_2012Metric_Pad1.15x1.40mm_HandSolder" H 7488 1350 50  0001 C CNN
+F 3 "~" H 7450 1500 50  0001 C CNN
+	1    7450 1500
+	-1   0    0    1
+$EndComp
+$Comp
+L Device:C C16
+U 1 1 5C4D029F
+P 7800 1500
+F 0 "C16" H 7700 1600 50  0000 C CNN
+F 1 "0.1 uF" H 7650 1400 50  0000 C CNN
+F 2 "Capacitor_SMD:C_0805_2012Metric_Pad1.15x1.40mm_HandSolder" H 7838 1350 50  0001 C CNN
+F 3 "~" H 7800 1500 50  0001 C CNN
+	1    7800 1500
+	-1   0    0    1
+$EndComp
+$Comp
+L Device:C C17
+U 1 1 5C4D02A5
+P 8150 1500
+F 0 "C17" H 8050 1600 50  0000 C CNN
+F 1 "0.1 uF" H 8000 1400 50  0000 C CNN
+F 2 "Capacitor_SMD:C_0805_2012Metric_Pad1.15x1.40mm_HandSolder" H 8188 1350 50  0001 C CNN
+F 3 "~" H 8150 1500 50  0001 C CNN
+	1    8150 1500
+	-1   0    0    1
+$EndComp
+Wire Wire Line
+	7100 1650 7100 1900
+Wire Wire Line
+	7100 1650 7450 1650
+Connection ~ 7100 1650
+Wire Wire Line
+	7450 1650 7800 1650
+Connection ~ 7450 1650
+Wire Wire Line
+	7800 1650 8150 1650
+Connection ~ 7800 1650
+Wire Wire Line
+	7100 1350 7450 1350
+Wire Wire Line
+	7450 1350 7800 1350
+Connection ~ 7450 1350
+Wire Wire Line
+	7800 1350 8150 1350
+Connection ~ 7800 1350
+$Comp
+L power:+3V3 #PWR022
+U 1 1 5C50EBF0
+P 7100 1200
+F 0 "#PWR022" H 7100 1050 50  0001 C CNN
+F 1 "+3V3" H 7115 1373 50  0000 C CNN
+F 2 "" H 7100 1200 50  0001 C CNN
+F 3 "" H 7100 1200 50  0001 C CNN
+	1    7100 1200
+	1    0    0    -1
+$EndComp
+Wire Wire Line
+	7100 1200 7100 1350
+Connection ~ 7100 1350
+Wire Wire Line
+	8800 1350 8800 1850
+Wire Wire Line
+	8700 2100 8700 1850
+Wire Wire Line
+	8700 1850 8800 1850
+Connection ~ 8800 1850
+Wire Wire Line
+	8800 1850 8800 2100
+Wire Wire Line
+	8600 2100 8600 1850
+Wire Wire Line
+	8600 1850 8700 1850
+Connection ~ 8700 1850
+Wire Wire Line
+	8900 2100 8900 1850
+Wire Wire Line
+	8900 1850 8800 1850
+Wire Wire Line
+	9000 2100 9000 1850
+Wire Wire Line
+	9000 1850 8900 1850
+Connection ~ 8900 1850
+$Comp
+L Device:C C18
+U 1 1 5C53AD8B
+P 8500 1500
+F 0 "C18" H 8400 1600 50  0000 C CNN
+F 1 "0.1 uF" H 8350 1400 50  0000 C CNN
+F 2 "Capacitor_SMD:C_0805_2012Metric_Pad1.15x1.40mm_HandSolder" H 8538 1350 50  0001 C CNN
+F 3 "~" H 8500 1500 50  0001 C CNN
+	1    8500 1500
+	-1   0    0    1
+$EndComp
+Wire Wire Line
+	8150 1650 8500 1650
+Wire Wire Line
+	8150 1350 8500 1350
+Connection ~ 8150 1350
+Connection ~ 8150 1650
+Wire Wire Line
+	8500 1350 8800 1350
+Connection ~ 8500 1350
 $EndSCHEMATC

Commit message: finalize LEDs: 0603 with 6.8 ohm resistors
Parts:
- D1, D2, D3, D4: footprint LED_SMD:LED_1206_3216Metric_Pad1.42x1.75mm_HandSolder -> LED_SMD:LED_0603_1608Metric_Pad1.05x0.95mm_HandSolder
- R2, R3, R4, R5: value R -> 6.8
Changed lines of the file:
@@
 F 0 "D1" H 7842 3145 50  0000 C CNN
 F 1 "LED" H 7842 3236 50  0000 C CNN
-F 2 "LED_SMD:LED_1206_3216Metric_Pad1.42x1.75mm_HandSolder" H 7850 3400 50  0001 C CNN
+F 2 "LED_SMD:LED_0603_1608Metric_Pad1.05x0.95mm_HandSolder" H 7850 3400 50  0001 C CNN
 F 3 "~" H 7850 3400 50  0001 C CNN
 	1    7850 3400
@@
 P 7550 3400
 F 0 "R2" V 7343 3400 50  0000 C CNN
-F 1 "R" V 7434 3400 50  0000 C CNN
+F 1 "6.8" V 7434 3400 50  0000 C CNN
 F 2 "Resistor_SMD:R_0805_2012Metric_Pad1.15x1.40mm_HandSolder" V 7480 3400 50  0001 C CNN
 F 3 "~" H 7550 3400 50  0001 C CNN
@@
 F 0 "D4" H 7842 4345 50  0000 C CNN
 F 1 "LED" H 7842 4436 50  0000 C CNN
-F 2 "LED_SMD:LED_1206_3216Metric_Pad1.42x1.75mm_HandSolder" H 7850 4600 50  0001 C CNN
+F 2 "LED_SMD:LED_0603_1608Metric_Pad1.05x0.95mm_HandSolder" H 7850 4600 50  0001 C CNN
 F 3 "~" H 7850 4600 50  0001 C CNN
 	1    7850 4600
@@
 P 7550 4600
 F 0 "R5" V 7343 4600 50  0000 C CNN
-F 1 "R" V 7434 4600 50  0000 C CNN
+F 1 "6.8" V 7434 4600 50  0000 C CNN
 F 2 "Resistor_SMD:R_0805_2012Metric_Pad1.15x1.40mm_HandSolder" V 7480 4600 50  0001 C CNN
 F 3 "~" H 7550 4600 50  0001 C CNN
@@
 F 0 "D2" H 7842 3545 50  0000 C CNN
 F 1 "LED" H 7842 3636 50  0000 C CNN
-F 2 "LED_SMD:LED_1206_3216Metric_Pad1.42x1.75mm_HandSolder" H 7850 3800 50  0001 C CNN
+F 2 "LED_SMD:LED_0603_1608Metric_Pad1.05x0.95mm_HandSolder" H 7850 3800 50  0001 C CNN
 F 3 "~" H 7850 3800 50  0001 C CNN
 	1    7850 3800
@@
 P 7550 3800
 F 0 "R3" V 7343 3800 50  0000 C CNN
-F 1 "R" V 7434 3800 50  0000 C CNN
+F 1 "6.8" V 7434 3800 50  0000 C CNN
 F 2 "Resistor_SMD:R_0805_2012Metric_Pad1.15x1.40mm_HandSolder" V 7480 3800 50  0001 C CNN
 F 3 "~" H 7550 3800 50  0001 C CNN
@@
 F 0 "D3" H 7842 3945 50  0000 C CNN
 F 1 "LED" H 7842 4036 50  0000 C CNN
-F 2 "LED_SMD:LED_1206_3216Metric_Pad1.42x1.75mm_HandSolder" H 7850 4200 50  0001 C CNN
+F 2 "LED_SMD:LED_0603_1608Metric_Pad1.05x0.95mm_HandSolder" H 7850 4200 50  0001 C CNN
 F 3 "~" H 7850 4200 50  0001 C CNN
 	1    7850 4200
@@
 P 7550 4200
 F 0 "R4" V 7343 4200 50  0000 C CNN
-F 1 "R" V 7434 4200 50  0000 C CNN
+F 1 "6.8" V 7434 4200 50  0000 C CNN
 F 2 "Resistor_SMD:R_0805_2012Metric_Pad1.15x1.40mm_HandSolder" V 7480 4200 50  0001 C CNN
 F 3 "~" H 7550 4200 50  0001 C CNN

Commit message: change VCC to 3V3 on SWD header
Connections:
- net labels removed: VCC
Changed lines of the file:
@@
 	3850 1100 4300 1100
 NoConn ~ 4300 1400
-$Comp
-L power:VCC #PWR0120
-U 1 1 5B9A1F01
-P 3850 850
-F 0 "#PWR0120" H 3850 700 50  0001 C CNN
-F 1 "VCC" H 3867 1023 50  0000 C CNN
-F 2 "" H 3850 850 50  0001 C CNN
-F 3 "" H 3850 850 50  0001 C CNN
-	1    3850 850
-	1    0    0    -1
-$EndComp
 Wire Wire Line
 	3850 850  3850 900
@@
 	8500 1350 8800 1350
 Connection ~ 8500 1350
+$Comp
+L power:+3V3 #PWR?
+U 1 1 5C3EDF8C
+P 3850 850
+F 0 "#PWR?" H 3850 700 50  0001 C CNN
+F 1 "+3V3" H 3865 1023 50  0000 C CNN
+F 2 "" H 3850 850 50  0001 C CNN
+F 3 "" H 3850 850 50  0001 C CNN
+	1    3850 850
+	1    0    0    -1
+$EndComp
 $EndSCHEMATC

Commit message: connect pin 6 of SWD header to GND
Connections:
- wire segments 152 -> 154
- no-connect marks 2 -> 1
Changed lines of the file:
@@
 L power:GND #PWR0119
 U 1 1 5B995EDB
-P 3850 1150
-F 0 "#PWR0119" H 3850 900 50  0001 C CNN
-F 1 "GND" H 3855 977 50  0000 C CNN
-F 2 "" H 3850 1150 50  0001 C CNN
-F 3 "" H 3850 1150 50  0001 C CNN
-	1    3850 1150
+P 3850 1500
+F 0 "#PWR0119" H 3850 1250 50  0001 C CNN
+F 1 "GND" H 3855 1327 50  0000 C CNN
+F 2 "" H 3850 1500 50  0001 C CNN
+F 3 "" H 3850 1500 50  0001 C CNN
+	1    3850 1500
 	1    0    0    -1
 $EndComp
@@
 $EndComp
 Wire Wire Line
-	3850 1150 3850 1100
+	3850 1500 3850 1400
 Wire Wire Line
 	3850 1100 4300 1100
-NoConn ~ 4300 1400
 Wire Wire Line
 	3850 850  3850 900
@@
 	1    0    0    -1
 $EndComp
+Wire Wire Line
+	4300 1400 3850 1400
+Connection ~ 3850 1400
+Wire Wire Line
+	3850 1400 3850 1100
 $EndSCHEMATC

Commit message: quadrant.sch: update for rev 3.1
reroute i2c lines to PB6/PB7
route VL6180x:GPIO0's to the MCU
move LED lines for convenience in routing
Connections:
- net labels added: EN1, EN2, EN3, EN4
- wire segments 154 -> 173

Commit message: update layout for rev 3.1
Parts:
- removed C11: 0.1 uF, Capacitor_SMD:C_0805_2012Metric_Pad1.15x1.40mm_HandSolder, symbol Device:C
Connections:
- wire segments 173 -> 171
Changed lines of the file:
@@
 L power:GND #PWR0103
 U 1 1 5C36188E
-P 7850 1850
-F 0 "#PWR0103" H 7850 1600 50  0001 C CNN
-F 1 "GND" H 7855 1677 50  0000 C CNN
-F 2 "" H 7850 1850 50  0001 C CNN
-F 3 "" H 7850 1850 50  0001 C CNN
-	1    7850 1850
-	1    0    0    -1
-$EndComp
-$Comp
-L Device:C C11
-U 1 1 5C361896
-P 7850 1450
-F 0 "C11" H 7750 1550 50  0000 C CNN
-F 1 "0.1 uF" H 7700 1350 50  0000 C CNN
-F 2 "Capacitor_SMD:C_0805_2012Metric_Pad1.15x1.40mm_HandSolder" H 7888 1300 50  0001 C CNN
-F 3 "~" H 7850 1450 50  0001 C CNN
-	1    7850 1450
-	-1   0    0    1
+P 8200 1850
+F 0 "#PWR0103" H 8200 1600 50  0001 C CNN
+F 1 "GND" H 8205 1677 50  0000 C CNN
+F 2 "" H 8200 1850 50  0001 C CNN
+F 3 "" H 8200 1850 50  0001 C CNN
+	1    8200 1850
+	1    0    0    -1
 $EndComp
 $Comp
@@
 $EndComp
 Wire Wire Line
-	7850 1600 7850 1850
-Wire Wire Line
-	7850 1600 8200 1600
-Connection ~ 7850 1600
+	8200 1600 8200 1850
 Wire Wire Line
 	8200 1600 8550 1600
-Connection ~ 8200 1600
 Wire Wire Line
 	8550 1600 8900 1600
 Connection ~ 8550 1600
 Wire Wire Line
-	7850 1300 8200 1300
-Wire Wire Line
 	8200 1300 8550 1300
-Connection ~ 8200 1300
 Wire Wire Line
 	8550 1300 8900 1300
@@
 L power:+3V3 #PWR022
 U 1 1 5C50EBF0
-P 7850 1150
-F 0 "#PWR022" H 7850 1000 50  0001 C CNN
-F 1 "+3V3" H 7865 1323 50  0000 C CNN
-F 2 "" H 7850 1150 50  0001 C CNN
-F 3 "" H 7850 1150 50  0001 C CNN
-	1    7850 1150
-	1    0    0    -1
-$EndComp
-Wire Wire Line
-	7850 1150 7850 1300
-Connection ~ 7850 1300
+P 8200 1150
+F 0 "#PWR022" H 8200 1000 50  0001 C CNN
+F 1 "+3V3" H 8215 1323 50  0000 C CNN
+F 2 "" H 8200 1150 50  0001 C CNN
+F 3 "" H 8200 1150 50  0001 C CNN
+	1    8200 1150
+	1    0    0    -1
+$EndComp
 Wire Wire Line
 	9550 1300 9550 1800
@@
 Wire Wire Line
 	2950 6450 2950 6550
+Connection ~ 8200 1600
+Wire Wire Line
+	8200 1150 8200 1300
+Connection ~ 8200 1300
 $EndSCHEMATC

Commit message: current-limiting resistors: 6.8 -> 10 ohm
Parts:
- R2, R3, R4, R5: value 6.8 -> 10
Changed lines of the file:
@@
 Sheet 1 1
 Title "Quadrant Board"
-Date "2019-02-09"
+Date "2019-03-04"
 Rev "3.1"
 Comp "Chris Chronopoulos"
@@
 P 8300 2950
 F 0 "R2" V 8093 2950 50  0000 C CNN
-F 1 "6.8" V 8184 2950 50  0000 C CNN
+F 1 "10" V 8184 2950 50  0000 C CNN
 F 2 "Resistor_SMD:R_0805_2012Metric_Pad1.15x1.40mm_HandSolder" V 8230 2950 50  0001 C CNN
 F 3 "~" H 8300 2950 50  0001 C CNN
@@
 P 8300 4850
 F 0 "R5" V 8093 4850 50  0000 C CNN
-F 1 "6.8" V 8184 4850 50  0000 C CNN
+F 1 "10" V 8184 4850 50  0000 C CNN
 F 2 "Resistor_SMD:R_0805_2012Metric_Pad1.15x1.40mm_HandSolder" V 8230 4850 50  0001 C CNN
 F 3 "~" H 8300 4850 50  0001 C CNN
@@
 P 8300 3350
 F 0 "R3" V 8093 3350 50  0000 C CNN
-F 1 "6.8" V 8184 3350 50  0000 C CNN
+F 1 "10" V 8184 3350 50  0000 C CNN
 F 2 "Resistor_SMD:R_0805_2012Metric_Pad1.15x1.40mm_HandSolder" V 8230 3350 50  0001 C CNN
 F 3 "~" H 8300 3350 50  0001 C CNN
@@
 P 8300 3750
 F 0 "R4" V 8093 3750 50  0000 C CNN
-F 1 "6.8" V 8184 3750 50  0000 C CNN
+F 1 "10" V 8184 3750 50  0000 C CNN
 F 2 "Resistor_SMD:R_0805_2012Metric_Pad1.15x1.40mm_HandSolder" V 8230 3750 50  0001 C CNN
 F 3 "~" H 8300 3750 50  0001 C CNN
